Commit message: rviz added, images added

File: anro2/urdf/fixed.urdf (robot description, URDF)
Before this commit: robot robot, 4 links, 3 joints
Links:
- removed link base_l
- added link base_link; visual box size=${box_size} ${box_size} ${urdf_data['i1']['l_len']}
Joints:
- removed joint base_link1
- added joint base_link_link1: type fixed, parent base_link, child link1, origin xyz=${urdf_data['i1']['j_xyz']} rpy=${urdf_data['i1']['j_rpy']}

File: anro2/urdf/wiggly.urdf (robot description, URDF)
Before this commit: robot robot, 4 links, 3 joints
Links:
- removed link base_l
- added link base_link; visual box size=${box_size} ${box_size} ${urdf_data['i1']['l_len']}
Joints:
- removed joint base_link1
- added joint base_link_link1: type prismatic, parent base_link, child link1, origin xyz=${urdf_data['i1']['j_xyz']} rpy=${urdf_data['i1']['j_rpy']}, axis 0 1 0, limit lower=0.0 upper=1 effort=1000.0 velocity=0.5

Commit message: bugs fixed

File: anro2/urdf/fixed.urdf (robot description, URDF)
Before this commit: robot robot, 4 links, 3 joints
Links:
- added link link4; visual cylinder length=${last_link_len} radius=${last_link_radius}
- link base_link: geometry visual box size=${base_box_size} ${base_box_size} ${base_box_size}
- link link1: geometry visual box size=${box_size} ${box_size} ${urdf_data['i1']['l_len']}
- link link2: geometry visual box size=${box_size} ${box_size} ${urdf_data['i2']['l_len']}
- link link3: geometry visual box size=${box_size} ${box_size} ${urdf_data['i2']['l_len']}
Joints:
- added joint link3_link4: type fixed, parent link3, child link4, origin xyz=${urdf_data['i3']['j_xyz']} rpy=${urdf_data['i3']['j_rpy']}
- joint base_link_link1: origin xyz=${urdf_data['i1']['j_xyz']} rpy=${urdf_data['i1']['j_rpy']} -> xyz=0 0 0 rpy=0 0 0
- joint link1_link2: origin xyz=${urdf_data['i2']['j_xyz']} rpy=${urdf_data['i2']['j_rpy']} -> xyz=${urdf_data['i1']['j_xyz']} rpy=${urdf_data['i1']['j_rpy']}
- joint link2_link3: origin xyz=${urdf_data['i3']['j_xyz']} rpy=${urdf_data['i3']['j_rpy']} -> xyz=${urdf_data['i2']['j_xyz']} rpy=${urdf_data['i2']['j_rpy']}

File: anro2/urdf/wiggly.urdf (robot description, URDF)
Before this commit: robot robot, 4 links, 3 joints
Links:
- added link link4; visual cylinder length=${last_link_len} radius=${last_link_radius}
- link base_link: geometry visual box size=${base_box_size} ${base_box_size} ${base_box_size}
- link link1: geometry visual box size=${box_size} ${box_size} ${urdf_data['i1']['l_len']}
- link link2: geometry visual box size=${box_size} ${box_size} ${urdf_data['i2']['l_len']}
- link link3: geometry visual box size=${box_size} ${box_size} ${urdf_data['i2']['l_len']}
Joints:
- added joint link3_link4: type fixed, parent link3, child link4, origin xyz=${urdf_data['i3']['j_xyz']} rpy=${urdf_data['i3']['j_rpy']}
- joint base_link_link1: axis 0 1 0 -> 0 0 1; limit lower=0.0 upper=1 effort=1000.0 velocity=0.5 -> lower=-1 upper=0 effort=1000.0 velocity=0.5; origin xyz=${urdf_data['i1']['j_xyz']} rpy=${urdf_data['i1']['j_rpy']} -> xyz=0 0 0 rpy=0 0 0
- joint link1_link2: axis 0 1 0 -> 0 0 1; limit lower=0.0 upper=1 effort=1000.0 velocity=0.5 -> lower=-1 upper=0 effort=1000.0 velocity=0.5; origin xyz=${urdf_data['i2']['j_xyz']} rpy=${urdf_data['i2']['j_rpy']} -> xyz=${urdf_data['i1']['j_xyz']} rpy=${urdf_data['i1']['j_rpy']}
- joint link2_link3: axis (none) -> 0 0 1; limit (none) -> lower=-1 upper=0 effort=1000.0 velocity=0.5; origin xyz=${urdf_data['i3']['j_xyz']} rpy=${urdf_data['i3']['j_rpy']} -> xyz=${urdf_data['i2']['j_xyz']} rpy=${urdf_data['i2']['j_rpy']}; type fixed -> prismatic
